File: Farfadet_differential_transceiver/Farfadet_differential_transceiver.kicad_pcb (KiCad board)
At the start: 2 copper layers, 19 x 36 mm, 16 parts, among them J1 Conn_01x05, J2 Conn_01x05, J3 XLR connector, J4 picoBlade connector, Q1 BSS84, U1 TXS0101DBV, U2 SP3485CN

Commit message: Differential transceiver : fix XLR connector pinout
Other:
- board text added: "T. Magnier v1.0b 06/2018"
- board text removed: "T. Magnier v1.0 01/2018"
Changed lines of the file:
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@@
     (links 40)
     (no_connects 0)
-    (area 121.224999 87.224999 171.35 142.200001)
+    (area 124.424999 90.424999 143.575001 126.575001)
     (thickness 1.6)
     (drawings 35)
@@
   (title_block
     (title "Farfadet - Differential transceiver for uC")
-    (date 2018-01-25)
-    (rev 1.0)
+    (date 2018-06-13)
+    (rev 1.0b)
     (company "Tom Magnier")
   )
@@
     )
   )
+  (module tom_kicad_lib:Solder_Jumper_2_conn (layer B.Cu)
+    (at 129.75 118.5)
+    (descr "Pontet Goute de soudure")
+    (solder_mask_margin 0.16)
+    (attr virtual)
+    (fp_text reference JP2 (at 2.25 -0.25 90) (layer B.SilkS)
+      (effects (font (size 1 1) (thickness 0.15)) (justify mirror))
+    )
+    (fp_text value Jumper_NC_Small (at 1.524 0 90) (layer B.Fab) hide
+      (effects (font (size 1 1) (thickness 0.15)) (justify mirror))
+    )
+    (fp_line (start 0 0.4) (end 0 -0.4) (layer B.Cu) (width 0.5))
+    (fp_line (start -0.889 1.27) (end -0.889 -1.27) (layer B.SilkS) (width 0.15))
+    (fp_line (start 0.889 -1.27) (end 0.889 1.27) (layer B.SilkS) (width 0.15))
+    (fp_line (start 0.889 -1.27) (end -0.889 -1.27) (layer B.SilkS) (width 0.15))
+    (fp_line (start -0.889 1.27) (end 0.889 1.27) (layer B.SilkS) (width 0.15))
+    (pad 1 smd rect (at 0 0.635) (size 1.27 0.9652) (layers B.Cu B.Mask)
+      (net 9 /1WIRE_DATA))
+    (pad 2 smd rect (at 0 -0.635) (size 1.27 0.9652) (layers B.Cu B.Mask)
+      (net 12 /RS485_A/1WIRE))
+  )
   (module tom_kicad_lib:Neutrik_XLR_NC3FAAH2 (layer F.Cu)
     (at 134 100)
@@
       (effects (font (size 0.8 0.8) (thickness 0.1)))
     )
-    (fp_text value "XLR connector" (at 0 0.75) (layer F.Fab) hide
+    (fp_text value "XLR connector" (at 0 0.75) (layer F.Fab)
       (effects (font (size 0.8 0.8) (thickness 0.1)))
     )
@@
     (pad 3 thru_hole circle (at 0 7.395) (size 2.4 2.4) (drill 1.2) (layers *.Cu *.Mask)
       (net 12 /RS485_A/1WIRE))
-    (pad 4 thru_hole circle (at -6.985 -1.495) (size 2.4 2.4) (drill 1.2) (layers *.Cu *.Mask)
+    (pad 4 thru_hole circle (at -8.25 -2.75) (size 2.4 2.4) (drill 1.2) (layers *.Cu *.Mask)
       (net 1 GND))
     (model /home/tom/Dropbox/kicad/3d/D-NC3FAAH2.wrl
@@
       (rotate (xyz 0 0 0))
     )
-  )
-  (module tom_kicad_lib:Solder_Jumper_2_conn (layer B.Cu)
-    (at 129.75 118.5)
-    (descr "Pontet Goute de soudure")
-    (solder_mask_margin 0.16)
-    (attr virtual)
-    (fp_text reference JP2 (at 2.25 -0.25 90) (layer B.SilkS)
-      (effects (font (size 1 1) (thickness 0.15)) (justify mirror))
-    )
-    (fp_text value Jumper_NC_Small (at 1.524 0 90) (layer B.Fab) hide
-      (effects (font (size 1 1) (thickness 0.15)) (justify mirror))
-    )
-    (fp_line (start 0 0.4) (end 0 -0.4) (layer B.Cu) (width 0.5))
-    (fp_line (start -0.889 1.27) (end -0.889 -1.27) (layer B.SilkS) (width 0.15))
-    (fp_line (start 0.889 -1.27) (end 0.889 1.27) (layer B.SilkS) (width 0.15))
-    (fp_line (start 0.889 -1.27) (end -0.889 -1.27) (layer B.SilkS) (width 0.15))
-    (fp_line (start -0.889 1.27) (end 0.889 1.27) (layer B.SilkS) (width 0.15))
-    (pad 1 smd rect (at 0 0.635) (size 1.27 0.9652) (layers B.Cu B.Mask)
-      (net 9 /1WIRE_DATA))
-    (pad 2 smd rect (at 0 -0.635) (size 1.27 0.9652) (layers B.Cu B.Mask)
-      (net 12 /RS485_A/1WIRE))
   )
   (gr_arc (start 126 125) (end 126 126.5) (angle 90) (layer Edge.Cuts) (width 0.15))
@@
     (effects (font (size 1 1) (thickness 0.2)) (justify left mirror))
   )
-  (gr_text "T. Magnier\nv1.0  01/2018" (at 143.25 109) (layer B.SilkS)
+  (gr_text "T. Magnier\nv1.0b 06/2018" (at 143.25 109) (layer B.SilkS)
     (effects (font (size 1 1) (thickness 0.2)) (justify left mirror))
   )
