File: Farfadet_magnetic_encoder_extension/Farfadet_magnetic_encoder_extension.kicad_pcb (KiCad board)
At the start: 2 copper layers, 58 x 58 mm, 24 parts, among them J1 Conn_02x05_Odd_Even, J2 Conn_01x02, J3 TEST_1P, U1 AS5132-HSS*

Commit message: Magnetic encoder extension v1.1 : add resistive voltage dividers on 5V signals
Parts:
- removed R2, R3: 4.7k, Resistors_SMD:R_0603
- added RN1: 4.7k, Resistors_SMD:R_Array_Convex_4x0603, B.Cu at (159.0, 110.2)
- added RN2: 4.7k, Resistors_SMD:R_Array_Convex_4x0603, B.Cu at (155.0, 110.2)
- D1: value LED_Small -> Red
- D2: value LED_Small -> Green
- moved J3 5.11 mm to (160.0, 104.5)
Connections:
- U1 pad 3: /ENCN -> Net-(RN2-Pad6)
- U1 pad 4: /ENCB -> Net-(RN2-Pad7)
- U1 pad 7: /ENCA -> Net-(RN1-Pad6)
Routing:
- net GND: track 81.1 -> 121.8 mm, vias 39 -> 44
- net Net-(RN1-Pad6): track 0.00 -> 13.0 mm
- net /SDO: track 17.5 -> 30.5 mm
- net /ENCA: track 18.5 -> 5.91 mm
- net /ENCB: track 16.8 -> 6.83 mm
- net /ENCN: track 15.6 -> 6.65 mm
- net Net-(RN2-Pad7): track 0.00 -> 8.64 mm
- net Net-(RN2-Pad6): track 0.00 -> 7.67 mm
- net Net-(J3-Pad1): track 8.06 -> 2.91 mm
- net /SCK: track 23.7 -> 28.5 mm
- net /~CS~_EXT: track 29.0 -> 32.9 mm
- net Net-(D2-Pad2): track 7.19 -> 9.84 mm
- net Net-(RN1-Pad8): track 4.10 -> 6.72 mm
- net Net-(RN1-Pad7): track 4.65 -> 5.39 mm
Other:
- board text added: "T. Magnier Rev 1.1 06/2018"
- board text removed: "T. Magnier Rev 1.0 01/2018"
